Commit message: Fixed some major issues
Added missing _'s and "'s and fixed other typos and mis-keying.

File: ros_ws/src/typepyt/urdf/typepyt.urdf.xacro (robot description, xacro)
@@ -1,4 +1,4 @@
 <?xml version="1.0"?>
-<robot name="typepyt">
+<robot xmlns:xacro="http://ros.org/wiki/xacro" name="typepyt">
   <xacro:macro name="box_inertial" params="x y z mass *origin">
     <inertial>
@@ -45,13 +45,13 @@
   <controller_plugin_gazebo />
   <!--world + base_link -->
-  <link name='world"/>
+  <link name="world" />
   <joint name="fixed" type="fixed">
-    <origin xyz="0.0 -0.4 0.0"/>
-    <parent link="world"/>
-    <child link="base_link"/>
+    <origin xyz="0.0 -0.4 0.0" />
+    <parent link="world" />
+    <child link="base_link" />
   </joint>
   <link name="base_link">
     <visual>
-      <origin xyz="0 -0.4 0"/>
+      <origin xyz="0 0 0"/>
       <geometry>
         <box size="0.95 1.425 0.2"/>
@@ -60,11 +60,11 @@
     </visual>
     <collision>
-      <origin xyz="0 -0.4 0"/>
+      <origin xyz="0 0 0"/>
       <geometry>
         <box size="0.95 1.425 0.2"/>
       </geometry>
     </collision>
-    <xacro:box_inertial mass="1.0" x="0.18" y="0.8" z="0.25>
-      <origin xyz="0 -0.4 0"/>
+    <xacro:box_inertial mass="1.0" x="0.18" y="0.8" z="0.25">
+      <origin xyz="0 0 0" />
     </xacro:box_inertial>
   </link>
@@ -95,5 +95,5 @@
       </geometry>
     </collision>
-    <xacro:box inertial mass="1.0" x="0.04" y="0.04" z="0.05">
+    <xacro:box_inertial mass="1.0" x="0.04" y="0.04" z="0.05">
       <origin xyz="0 0 0.25"/>
     </xacro:box_inertial>
@@ -121,5 +121,5 @@
     <dynamics damping="0.05" friction="0.0" />
   </joint>
-  <link name="upper arm">
+  <link name="upper_arm">
     <visual>
       <origin xyz="0 0 0.4"/>
@@ -135,5 +135,5 @@
       </geometry>
     </collision>
-    <xacro:box inertial mass="1.0" x="0.16" y="0.16" z="0.32">
+    <xacro:box_inertial mass="1.0" x="0.16" y="0.16" z="0.32">
       <origin xyz="0 0 0"/>
     </xacro:box_inertial>
@@ -153,8 +153,8 @@
   <!-- upper_arm + upper_arm1 -->
   <joint name="elbow" type="revolute">
-    <origin xyz="0 0 0.8" rpy="0 3.36 0"/>
-    <parent link="upper_arm"/>
-    <child link="upper_arm1/>
-    <axis xyz="0 0 0"/>
+    <origin xyz="0 0 0.8" rpy="0 3.36 0" />
+    <parent link="upper_arm" />
+    <child link="upper_arm1" />
+    <axis xyz="0 0 0.8"/>
     <limit lower="0.0" upper="0.0" velocity="0.0" effort="0.0" />
     <dynamics damping="0.0" friction="0.0" />
@@ -177,5 +177,5 @@
       </geometry>
     </collision>
-    <xacro:box inertial mass="1.0" x="0.04" y="0.04" z="0.05">
+    <xacro:box_inertial mass="1.0" x="0.04" y="0.04" z="0.05">
       <origin xyz="0.05 0.05 0.01"/>
     </xacro:box_inertial>
@@ -207,5 +207,5 @@
       </geometry>
     </collision>
-    <xacro:box inertial mass="1.0" x="0.16" y="0.16" z="0.32">
+    <xacro:box_inertial mass="1.0" x="0.16" y="0.16" z="0.32">
       <origin xyz="0 0 0.4"/>
     </xacro:box_inertial>
@@ -247,5 +247,5 @@
       </geometry>
     </collision>
-    <xacro:box inertial mass="1.0" x="0.0004" y="0.0004" z="0.002">
+    <xacro:box_inertial mass="1.0" x="0.0004" y="0.0004" z="0.002">
       <origin xyz="0 0 0"/>
     </xacro:box_inertial>
@@ -272,3 +272,3 @@
     </plugin>
   </gazebo>
-</robot
+</robot>

Commit message: Changed the model settings
Fixed problems with mimic joints not working in RVIZ--Haven't got it to work in Gazebo yet.

File: ros_ws/src/typepyt/urdf/typepyt.urdf.xacro (robot description, xacro)
@@ -47,5 +47,5 @@
   <link name="world" />
   <joint name="fixed" type="fixed">
-    <origin xyz="0.0 -0.4 0.0" />
+    <origin xyz="0.0 0.0 0.0" />
     <parent link="world" />
     <child link="base_link" />
@@ -74,5 +74,5 @@
   <!-- base_link + torso -->
   <joint name="hip" type="revolute">
-    <origin xyz="0 0 0.25" rpy="0 0 0"/>
+    <origin xyz="0 0 0.12" rpy="0 0 0"/>
     <parent link="base_link"/>
     <child link="torso"/>
@@ -114,8 +114,8 @@
   <!-- torso + upper_arm -->
   <joint name="shoulder" type="revolute">
-    <origin xyz="0.2 0 0.3" rpy="0 -1.57 0"/>
+    <origin xyz="0.2 0 0.3" rpy="0 -1.5708 0"/>
     <parent link="torso"/>
     <child link="upper_arm"/>
-    <axis xyz="0 0 0.4"/>
+    <axis xyz="0 1 0"/>
     <limit lower="0.52" upper="2.79" velocity="1.0" effort="30.0" />
     <dynamics damping="0.05" friction="0.0" />
@@ -144,5 +144,6 @@
   <transmission name="tran1">
     <type>transmission_interface/SimpleTransmission</type>
-    <joint name="shoulder">             <hardwareInterface>hardware_interface/PositionJointInterface</hardwareInterface>
+    <joint name="shoulder">
+      <hardwareInterface>hardware_interface/PositionJointInterface</hardwareInterface>
     </joint>
     <actuator name="motor1">
@@ -156,14 +157,15 @@
     <parent link="upper_arm" />
     <child link="upper_arm1" />
-    <axis xyz="0 0 0.8"/>
-    <limit lower="0.0" upper="0.0" velocity="0.0" effort="0.0" />
+    <axis xyz="0 -1 0"/>
+    <limit lower="0.87" upper="2.44" velocity="1.0" effort="30.0" />
+    <mimic joint="shoulder" multiplier="1" offset="0" />
     <dynamics damping="0.0" friction="0.0" />
   </joint>
   <xacro:mimic_joint_plugin_gazebo name_prefix="elbow"
-    parent_joint="fixed" mimic_joint="elbow"
+    parent_joint="shoulder" mimic_joint="elbow"
     has_pid="true" multiplier="1.0" max_effort="10.0" />
   <link name="upper_arm1">
     <visual>
-      <origin xyz="0.05 0.05 0.01"/>
+      <origin xyz="0 0 0.04"/>
       <geometry>
         <box size="0.05 0.05 0.01"/>
